Commit message: Add propellers' dae files

File: models/util/multirotor_base.urdf.xacro (robot description, xacro)
@@ -111,5 +111,5 @@
         <geometry>
           <!-- <cylinder length="0.005" radius="${radius_rotor}"/> --> <!-- [m] -->
-          <mesh filename="package://ardupilot_gazebo/models/util/propeller_${direction}.dae"
+          <mesh filename="package://marcus_gazebo/models/util/propeller_${direction}.dae"
             scale="${prop_scale} ${prop_scale} ${prop_scale}" />
           <!-- <box size="${2*radius_rotor} 0.01 0.005"/> -->
